File: hardware/takoyaki8.kicad_sch (KiCad schematic)
At the start: 0 parts

Commit message: Add key matrix and LED chain to schematic (wip)
Parts:
- added C1, C2, C3, C4: 100nF, Capacitor_SMD:C_0603_1608Metric, symbol Device:C
- added D1, D2, D3, D4, D5, D6, D7, D8: 1N4148W, Diode_SMD:D_SOD-123, symbol Device:D
- added LED1, LED2, LED3, LED4: WS2812B, LED_SMD:LED_WS2812B_PLCC4_5.0x5.0mm_P3.2mm, symbol LED:WS2812B
- added R1: 0R, Resistor_SMD:R_0603_1608Metric, symbol Device:R
- added SW1, SW2, SW3, SW4, SW5, SW6, SW7, SW8: SW_Push, takoyaki8:SW_choc_v2_HS_CPG135001S30_1u, symbol Switch:SW_Push
Connections:
- new net: D8.2 (A), SW8.2
- new net: D3.2 (A), SW3.2
- new net: D1.2 (A), SW1.2
- new net: D5.2 (A), SW5.2
- new net: LED1.4 (DIN), R1.2
- new net: D6.2 (A), SW6.2
- new net: D4.2 (A), SW4.2
- new net: D2.2 (A), SW2.2
- new net: D7.2 (A), SW7.2
- new net +5V: C1.1, C2.1, C3.1, C4.1, LED1.1 (VDD), LED2.1 (VDD), LED3.1 (VDD), LED4.1 (VDD)
- new net COL0: SW1.1, SW5.1
- new net COL1: SW2.1, SW6.1
- new net COL2: SW3.1, SW7.1
- new net COL3: SW4.1, SW8.1
- new net GND: C1.2, C2.2, C3.2, C4.2, LED1.3 (VSS), LED2.3 (VSS), LED3.3 (VSS), LED4.3 (VSS)
- new net LED_D1: LED1.2 (DOUT), LED2.4 (DIN)
- new net LED_D2: LED2.2 (DOUT), LED3.4 (DIN)
- new net LED_D3: LED3.2 (DOUT), LED4.4 (DIN)
- new net LED_DATA: R1.1
- new net ROW0: D1.1 (K), D2.1 (K), D3.1 (K), D4.1 (K)
- new net ROW1: D5.1 (K), D6.1 (K), D7.1 (K), D8.1 (K)
- no-connect marks 0 -> 2

Commit message: Add RP2040-Zero symbol and castellated footprint (provisional pads)
Parts:
- added U1: RP2040-Zero, takoyaki8:RP2040-Zero_Castellated, symbol takoyaki8:RP2040-Zero
Changed lines of the file:
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@@
+	)
+	(symbol
+		(lib_id "takoyaki8:RP2040-Zero")
+		(at 53.34 76.2 0)
+		(unit 1)
+		(body_style 1)
+		(exclude_from_sim no)
+		(in_bom yes)
+		(on_board yes)
+		(in_pos_files yes)
+		(dnp no)
+		(fields_autoplaced yes)
+		(property "Reference" "U1"
+			(at 53.34 58.42 0)
+			(show_name no)
+			(do_not_autoplace no)
+			(effects
+				(font
+					(size 1.27 1.27)
+				)
+			)
+		)
+		(property "Value" "RP2040-Zero"
+			(at 53.34 60.96 0)
+			(show_name no)
+			(do_not_autoplace no)
+			(effects
+				(font
+					(size 1.27 1.27)
+				)
+			)
+		)
+		(property "Footprint" "takoyaki8:RP2040-Zero_Castellated"
+			(at 53.34 76.2 0)
+			(hide yes)
+			(show_name no)
+			(do_not_autoplace no)
+			(effects
+				(font
+					(size 1.27 1.27)
+				)
+			)
+		)
+		(property "Datasheet" "https://www.waveshare.com/wiki/RP2040-Zero"
+			(at 53.34 76.2 0)
+			(hide yes)
+			(show_name no)
+			(do_not_autoplace no)
+			(effects
+				(font
+					(size 1.27 1.27)
+				)
+			)
+		)
+		(property "Description" "Waveshare RP2040-Zero module, castellated edge pins only. Pin numbers: left 1-9, bottom 10-14, right 15-23"
+			(at 53.34 76.2 0)
+			(hide yes)
+			(show_name no)
+			(do_not_autoplace no)
+			(effects
+				(font
+					(size 1.27 1.27)
+				)
+			)
+		)
+		(pin "16"
+		)
+		(pin "17"
+		)
+		(pin "11"
+		)
+		(pin "14"
+		)
+		(pin "15"
+		)
+		(pin "10"
+		)
+		(pin "13"
+		)
+		(pin "12"
+		)
+		(pin "9"
+		)
+		(pin "8"
+		)
+		(pin "7"
+		)
+		(pin "6"
+		)
+		(pin "1"
+		)
+		(pin "4"
+		)
+		(pin "5"
+		)
+		(pin "3"
+		)
+		(pin "2"
+		)
+		(pin "23"
+		)
+		(pin "22"
+		)
+		(pin "21"
+		)
+		(pin "20"
+		)
+		(pin "19"
+		)
+		(pin "18"
+		)
+		(instances
+			(project "takoyaki8"
+				(path "/7b50840c-3526-4ae7-981f-323960f4fcc3"
+					(reference "U1")
+					(unit 1)
+				)
+			)
+		)
 	)
 	(symbol

Commit message: Complete minimal schematic: matrix, LED chain, RP2040-Zero, OLED connector (ERC clean)
Parts:
- added J1: OLED_0.91in, Connector_PinHeader_2.54mm:PinHeader_1x04_P2.54mm_Vertical, symbol Connector_Generic:Conn_01x04
Connections:
- net +5V: now also U1.1 (5V)
- net COL0: now also U1.21 (GP2)
- net COL1: now also U1.20 (GP3)
- net COL2: now also U1.19 (GP4)
- net COL3: now also U1.18 (GP5)
- net GND: now also U1.2 (GND), J1.1 (Pin_1)
- net LED_DATA: now also U1.7 (GP26)
- net ROW0: now also U1.23 (GP0)
- net ROW1: now also U1.22 (GP1)
- net +3V3: now reaches U1.3 (3V3)
- net +3V3: now also J1.2 (Pin_2)
- net I2C_SCL: now reaches U1.8 (GP15)
- net I2C_SCL: now also J1.3 (Pin_3)
- net I2C_SDA: now reaches U1.9 (GP14)
- net I2C_SDA: now also J1.4 (Pin_4)
- no-connect marks 2 -> 12
Other:
- moved on the sheet: C1, C2, C3, C4, LED1, LED2, LED3, LED4, R1

Commit message: Add OLED header and flipped RP2040-Zero footprints (sandwich plan, provisional)
Parts:
- J1: footprint Connector_PinHeader_2.54mm:PinHeader_1x04_P2.54mm_Vertical -> takoyaki8:OLED_0.91in_I2C_Header
Changed lines of the file:
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@@
 			)
 		)
-		(property "Footprint" "Connector_PinHeader_2.54mm:PinHeader_1x04_P2.54mm_Vertical"
+		(property "Footprint" "takoyaki8:OLED_0.91in_I2C_Header"
 			(at 45.72 134.62 0)
 			(hide yes)

Commit message: Update flipped RP2040-Zero footprint: component zones from 1:1 print, larger window
Parts:
- U1: footprint takoyaki8:RP2040-Zero_Castellated -> takoyaki8:RP2040-Zero_Castellated_Flipped
Changed lines of the file:
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@@
 			)
 		)
-		(property "Footprint" "takoyaki8:RP2040-Zero_Castellated"
+		(property "Footprint" "takoyaki8:RP2040-Zero_Castellated_Flipped"
 			(at 53.34 76.2 0)
 			(hide yes)
