File: hardware/takoyaki8.kicad_pcb (KiCad board)
At the start: 2 copper layers, 99.9 x 82.1 mm, 33 parts, among them J1 OLED_0.91in, SW1 SW_Push, SW2 SW_Push, SW3 SW_Push, SW4 SW_Push, SW5 SW_Push, SW6 SW_Push, SW7 SW_Push, SW8 SW_Push, U1 RP2040-Zero

Commit message: Add silkscreen: logo, copyright, board name/rev, GitHub URL (DRC: 0 errors, 0 unconnected, 24 mouse-bite hole warnings)
Parts:
- added G***: LOGO, takoyaki8:TakoyaKeeb_logo, B.Cu at (113.5, 88.5)
Other:
- board text added: "github.com/takoyakeeb/takoyaki8"
- board text added: "takoyaki8 rev1.0"
- board text added: "© 2026 TakoyaKeeb"
